File: Hardware/SmallScalePrototype/PCB/clock.brd (EAGLE design)
At the start: 160 x 100 mm, 21 parts

Commit message: All wires routed, passing OSHPark DRC!
Routing:
- net VCC: track 155.9 -> 320.9 mm, vias 0 -> 4
- net LE: track 0.00 -> 155.0 mm, vias 0 -> 9
- net CLK: track 0.00 -> 137.8 mm, vias 0 -> 11
- net SDI3: track 0.00 -> 24.3 mm
- net SDI1: track 0.00 -> 24.3 mm
- net SDI4: track 0.00 -> 13.3 mm
- net SDI2: track 0.00 -> 9.52 mm
- net SDI0: track 0.00 -> 9.10 mm
- net SDI5: track 22.1 -> 24.3 mm
- net SDI7: track 22.1 -> 23.9 mm

Commit message: Centered displays, added mounting holes
Parts:
- moved U$2 5.08 mm to (97.8, 12.7)
- moved R3 5.08 mm to (66.0, 20.3)
- moved U$5 5.08 mm to (55.9, 12.7)
- moved R6 5.08 mm to (35.6, 20.3)
- moved U$7 5.08 mm to (29.2, 12.7)
- moved R8 5.08 mm to (8.89, 20.3)
- moved U$8 5.08 mm to (14.0, 12.7)
- moved DIS1 5.08 mm to (105.4, 12.7)
- moved DIS2 5.08 mm to (78.7, 12.7)
- moved DIS3 5.08 mm to (48.3, 12.7)
- moved DIS4 5.08 mm to (21.6, 12.7)
- moved R1 5.08 mm to (118.1, 4.45)
- moved R2 5.08 mm to (91.4, 4.45)
- moved R4 5.08 mm to (61.0, 4.45)
- moved R5 5.08 mm to (92.7, 20.3)
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Other:
- board outline removed

Commit message: minor brd tweaks
Parts:
- renumbered U$1 to SR1, U$2 to SR2, U$3 to SR3, U$4 to SR4, U$5 to SR5, U$6 to SR6, U$7 to SR7, U$8 to SR8
