File: Hardware/SmallScalePrototype/PCB/clock.sch (EAGLE design)
At the start: 12 parts

Commit message: Schematic v1
I think thats everything....
Parts:
- added R1, R2, R3, R4, R5, R6, R7, R8: (no value), resistor:R-US_R0603
- added SV1: (no value), con-lsta:FE05-1
Connections:
- new net CLK: SV1.3, U$1.CLK, U$2.CLK, U$3.CLK, U$4.CLK, U$5.CLK, U$6.CLK, U$7.CLK, U$8.CLK
- new net GND: R1.1, R2.1, R4.1, R7.1, SV1.1, U$1.GND, U$1.OE, U$3.GND, U$3.OE, U$5.GND, U$5.OE, U$7.GND, U$7.OE
- new net LE: SV1.2, U$1.LE(ED1), U$2.LE(ED1), U$3.LE(ED1), U$4.LE(ED1), U$5.LE(ED1), U$6.LE(ED1), U$7.LE(ED1), U$8.LE(ED1)
- new net N$11: R5.2, U$2.R_EXT
- new net N$15: R1.2, U$1.R_EXT
- new net N$16: R6.2, U$6.R_EXT
- new net N$17: R4.2, U$5.R_EXT
- new net N$18: R6.1, U$6.GND, U$6.OE
- new net N$19: R5.1, U$2.GND, U$2.OE
- new net N$24: R8.2, U$8.R_EXT
- new net N$25: R7.2, U$7.R_EXT
- new net N$26: R8.1, U$8.GND, U$8.OE
- new net N$7: R3.2, U$4.R_EXT
- new net ONES0: DIS1.A2, U$2.OUT0
- new net ONES1: DIS1.B2, U$2.OUT1
- new net ONES10: DIS2.D2, U$4.OUT3
- new net ONES11: DIS2.E2, U$4.OUT4
- new net ONES12: DIS2.F2, U$4.OUT5
- new net ONES13: DIS2.G2, U$4.OUT6
- new net ONES14: DIS3.A2, U$6.OUT0
- new net ONES15: DIS3.B2, U$6.OUT1
- new net ONES16: DIS3.C2, U$6.OUT2
- new net ONES17: DIS3.D2, U$6.OUT3
- new net ONES18: DIS3.E2, U$6.OUT4
- new net ONES19: DIS3.F2, U$6.OUT5
- new net ONES2: DIS1.C2, U$2.OUT2
- new net ONES20: DIS3.G2, U$6.OUT6
- new net ONES21: DIS4.A2, U$8.OUT0
- new net ONES22: DIS4.B2, U$8.OUT1
- new net ONES23: DIS4.C2, U$8.OUT2
- new net ONES24: DIS4.D2, U$8.OUT3
- new net ONES25: DIS4.E2, U$8.OUT4
- new net ONES26: DIS4.F2, U$8.OUT5
- new net ONES27: DIS4.G2, U$8.OUT6
- new net ONES3: DIS1.D2, U$2.OUT3
- new net ONES4: DIS1.E2, U$2.OUT4
- new net ONES5: DIS1.F2, U$2.OUT5
- new net ONES6: DIS1.G2, U$2.OUT6
- new net ONES7: DIS2.A2, U$4.OUT0
- new net ONES8: DIS2.B2, U$4.OUT1
- new net ONES9: DIS2.C2, U$4.OUT2
- new net SDI: SV1.4, U$1.SDI
- new net TENS0: DIS1.A1, U$1.OUT0
- new net TENS1: DIS1.B1, U$1.OUT1
- new net TENS10: DIS2.D1, U$3.OUT3
- new net TENS11: DIS2.C1, U$3.OUT2
- new net TENS12: DIS2.B1, U$3.OUT1
- new net TENS13: DIS2.A1, U$3.OUT0
- new net TENS14: DIS3.G1, U$5.OUT6
- new net TENS15: DIS3.F1, U$5.OUT5
- new net TENS16: DIS3.E1, U$5.OUT4
- new net TENS17: DIS3.D1, U$5.OUT3
- new net TENS18: DIS3.C1, U$5.OUT2
- new net TENS19: DIS3.B1, U$5.OUT1
- new net TENS2: DIS1.C1, U$1.OUT2
- new net TENS20: DIS3.A1, U$5.OUT0
- new net TENS21: DIS4.G1, U$7.OUT6
- new net TENS22: DIS4.F1, U$7.OUT5
- new net TENS23: DIS4.E1, U$7.OUT4
- new net TENS24: DIS4.D1, U$7.OUT3
- new net TENS25: DIS4.C1, U$7.OUT2
- new net TENS26: DIS4.B1, U$7.OUT1
- new net TENS27: DIS4.A1, U$7.OUT0
- new net TENS3: DIS1.D1, U$1.OUT3
- new net TENS4: DIS1.E1, U$1.OUT4
- new net TENS5: DIS1.F1, U$1.OUT5
- new net TENS6: DIS1.G1, U$1.OUT6
- new net TENS7: DIS2.G1, U$3.OUT6
- new net TENS8: DIS2.F1, U$3.OUT5
- new net TENS9: DIS2.E1, U$3.OUT4
- new net VCC: DIS1.CA1, DIS1.CA2, DIS2.CA1, DIS2.CA2, DIS3.CA1, DIS3.CA2, DIS4.CA1, DIS4.CA2, SV1.5, U$1.VDD, U$2.VDD, U$3.VDD, U$4.VDD, U$5.VDD, U$6.VDD, U$7.VDD, U$8.VDD
- net N$8: now also R2.2, U$3.R_EXT; no longer U$1.GND, U$2.GND, U$3.GND, U$4.GND, U$5.GND, U$6.GND, U$7.GND, U$8.GND
- net N$9: now also R3.1, U$4.GND, U$4.OE; no longer U$1.VDD, U$2.VDD, U$3.VDD, U$4.VDD, U$5.VDD, U$6.VDD, U$7.VDD, U$8.VDD
Other:
- moved on the sheet: DIS1, DIS2, DIS3, DIS4, U$1, U$2, U$3, U$4, U$5, U$6, U$7, U$8

Commit message: Fixed ERC warning
Connections:
- net N$1 renamed SDI1
- net N$10 renamed SDI3
- net N$14 renamed SDI2
- net N$20 renamed SDI5
- net N$23 renamed SDI4
- net N$27 renamed SDI7
- net N$30 renamed SDI6
- net ONES0 renamed DAYSONES0
- net ONES1 renamed DAYSONES1
- net ONES10 renamed HOURSONES3
- net ONES11 renamed HOURSONES4
- net ONES12 renamed HOURSONES5
- net ONES13 renamed HOURSONES6
- net ONES14 renamed MINUTESONES0
- net ONES15 renamed MINUTESONES1
- net ONES16 renamed MINUTESONES2
- net ONES17 renamed MINUTESONES3
- net ONES18 renamed MINUTESONES4
- net ONES19 renamed MINUTESONES5
- net ONES2 renamed DAYSONES2
- net ONES20 renamed MINUTESONES6
- net ONES21 renamed SECONDSONES0
- net ONES22 renamed SECONDSONES1
- net ONES23 renamed SECONDSONES2
- net ONES24 renamed SECONDSONES3
- net ONES25 renamed SECONDSONES4
- net ONES26 renamed SECONDSONES5
- net ONES27 renamed SECONDSONES6
- net ONES3 renamed DAYSONES3
- net ONES4 renamed DAYSONES4
- net ONES5 renamed DAYSONES5
- net ONES6 renamed DAYSONES6
- net ONES7 renamed HOURSONES0
- net ONES8 renamed HOURSONES1
- net ONES9 renamed HOURSONES2
- net SDI renamed SDI0
- net TENS0 renamed DAYSTENS0
- net TENS1 renamed DAYSTENS1
- net TENS10 renamed HOURSTENS3
- net TENS11 renamed HOURSTENS2
- net TENS12 renamed HOURSTENS1
- net TENS13 renamed HOURSTENS0
- net TENS14 renamed MINUTESTENS6
- net TENS15 renamed MINUTESTENS5
- net TENS16 renamed MINUTESTENS4
- net TENS17 renamed MINUTESTENS3
- net TENS18 renamed MINUTESTENS2
- net TENS19 renamed MINUTESTENS1
- net TENS2 renamed DAYSTENS2
- net TENS20 renamed MINUTESTENS0
- net TENS21 renamed SECONDSTENS6
- net TENS22 renamed SECONDSTENS5
- net TENS23 renamed SECONDSTENS4
- net TENS24 renamed SECONDSTENS3
- net TENS25 renamed SECONDSTENS2
- net TENS26 renamed SECONDSTENS1
- net TENS27 renamed SECONDSTENS0
- net TENS3 renamed DAYSTENS3
- net TENS4 renamed DAYSTENS4
- net TENS5 renamed DAYSTENS5
- net TENS6 renamed DAYSTENS6
- net TENS7 renamed HOURSTENS6
- net TENS8 renamed HOURSTENS5
- net TENS9 renamed HOURSTENS4
- removed net N$18: R6.1, U$6.GND, U$6.OE
- removed net N$19: R5.1, U$2.GND, U$2.OE
- removed net N$26: R8.1, U$8.GND, U$8.OE
- removed net N$9: R3.1, U$4.GND, U$4.OE
- net GND: now also R3.1, R5.1, R6.1, R8.1, U$2.GND, U$2.OE, U$4.GND, U$4.OE, U$6.GND, U$6.OE, U$8.GND, U$8.OE

Commit message: Most of the board work
Connections:
- net DAYSONES0: now also U$2.OUT6; no longer U$2.OUT0
- net DAYSONES1: now also U$2.OUT7; no longer U$2.OUT1
- net DAYSONES2: now also U$2.OUT0; no longer U$2.OUT2
- net DAYSONES3: now also U$2.OUT2; no longer U$2.OUT3
- net DAYSONES4: now also U$2.OUT3; no longer U$2.OUT4
- net DAYSONES6: now also U$2.OUT1; no longer U$2.OUT6
- net DAYSTENS0: now also U$1.OUT2; no longer U$1.OUT0
- net DAYSTENS1: now also U$1.OUT3; no longer U$1.OUT1
- net DAYSTENS2: now also U$1.OUT5; no longer U$1.OUT2
- net DAYSTENS3: now also U$1.OUT6; no longer U$1.OUT3
- net DAYSTENS4: now also U$1.OUT7; no longer U$1.OUT4
- net DAYSTENS5: now also U$1.OUT0; no longer U$1.OUT5
- net DAYSTENS6: now also U$1.OUT1; no longer U$1.OUT6
- net HOURSONES0: now also U$4.OUT6; no longer U$4.OUT0
- net HOURSONES1: now also U$4.OUT7; no longer U$4.OUT1
- net HOURSONES2: now also U$4.OUT0; no longer U$4.OUT2
- net HOURSONES3: now also U$4.OUT2; no longer U$4.OUT3
- net HOURSONES4: now also U$4.OUT3; no longer U$4.OUT4
- net HOURSONES6: now also U$4.OUT1; no longer U$4.OUT6
- net HOURSTENS0: now also U$3.OUT2; no longer U$3.OUT0
- net HOURSTENS1: now also U$3.OUT3; no longer U$3.OUT1
- net HOURSTENS2: now also U$3.OUT5; no longer U$3.OUT2
- net HOURSTENS3: now also U$3.OUT6; no longer U$3.OUT3
- net HOURSTENS4: now also U$3.OUT7; no longer U$3.OUT4
- net HOURSTENS5: now also U$3.OUT0; no longer U$3.OUT5
- net HOURSTENS6: now also U$3.OUT1; no longer U$3.OUT6
- net MINUTESONES0: now also U$6.OUT6; no longer U$6.OUT0
- net MINUTESONES1: now also U$6.OUT7; no longer U$6.OUT1
- net MINUTESONES2: now also U$6.OUT0; no longer U$6.OUT2
- net MINUTESONES3: now also U$6.OUT2; no longer U$6.OUT3
- net MINUTESONES4: now also U$6.OUT3; no longer U$6.OUT4
- net MINUTESONES6: now also U$6.OUT1; no longer U$6.OUT6
- net MINUTESTENS0: now also U$5.OUT2; no longer U$5.OUT0
- net MINUTESTENS1: now also U$5.OUT3; no longer U$5.OUT1
- net MINUTESTENS2: now also U$5.OUT5; no longer U$5.OUT2
- net MINUTESTENS3: now also U$5.OUT6; no longer U$5.OUT3
- net MINUTESTENS4: now also U$5.OUT7; no longer U$5.OUT4
- net MINUTESTENS5: now also U$5.OUT0; no longer U$5.OUT5
- net MINUTESTENS6: now also U$5.OUT1; no longer U$5.OUT6
- net SECONDSONES0: now also U$8.OUT6; no longer U$8.OUT0
- net SECONDSONES1: now also U$8.OUT7; no longer U$8.OUT1
- net SECONDSONES2: now also U$8.OUT0; no longer U$8.OUT2
- net SECONDSONES3: now also U$8.OUT2; no longer U$8.OUT3
- net SECONDSONES4: now also U$8.OUT3; no longer U$8.OUT4
- net SECONDSONES6: now also U$8.OUT1; no longer U$8.OUT6
- net SECONDSTENS0: now also U$7.OUT2; no longer U$7.OUT0
- net SECONDSTENS1: now also U$7.OUT3; no longer U$7.OUT1
- net SECONDSTENS2: now also U$7.OUT5; no longer U$7.OUT2
- net SECONDSTENS3: now also U$7.OUT6; no longer U$7.OUT3
- net SECONDSTENS4: now also U$7.OUT7; no longer U$7.OUT4
- net SECONDSTENS5: now also U$7.OUT0; no longer U$7.OUT5
- net SECONDSTENS6: now also U$7.OUT1; no longer U$7.OUT6

Commit message: minor brd tweaks
Parts:
- renumbered U$1 to SR1, U$2 to SR2, U$3 to SR3, U$4 to SR4, U$5 to SR5, U$6 to SR6, U$7 to SR7, U$8 to SR8
